File: ecg.sch (KiCad schematic (older format))
At the start: 25 parts, among them J1 Conn_01x01_Male, J2 Conn_01x01_Male, U1 TL072, U2 TL072

Commit message: work in progress pcb layout
Parts:
- removed J1, J2: Conn_01x01_Male, symbol Connector:Conn_01x01_Male
- added C107: C, Capacitor_THT:C_Rect_L7.2mm_W4.5mm_P5.00mm_FKS2_FKP2_MKS2_MKP2, symbol Device:C
- added C108: CP, Capacitor_THT:CP_Radial_D7.5mm_P2.50mm, symbol Device:CP
- added C109, C111, C6, C8: 100n, Capacitor_THT:C_Rect_L7.2mm_W4.5mm_P5.00mm_FKS2_FKP2_MKS2_MKP2, symbol Device:C
- added C110, C112, C5, C7: 47u, Capacitor_THT:CP_Radial_D7.5mm_P2.50mm, symbol Device:CP
- added JP1, JP11, JP2, JP22, JP3, JP33, JP4, JP44: Jumper, Connector_PinHeader_1.27mm:PinHeader_1x02_P1.27mm_Vertical, symbol Device:Jumper
- added R11: Rg1, Resistor_THT:R_Axial_DIN0207_L6.3mm_D2.5mm_P10.16mm_Horizontal, symbol Device:R
- added R12: Rg2, Resistor_THT:R_Axial_DIN0207_L6.3mm_D2.5mm_P10.16mm_Horizontal, symbol Device:R
- added RV1: R_POT, Potentiometer_THT:Potentiometer_Piher_PT-6-V_Vertical, symbol Device:R_POT
- added TP1: LowPass IN, Connector_PinHeader_1.27mm:PinHeader_1x01_P1.27mm_Vertical, symbol Connector:TestPoint
- added TP2: HighPass IN, Connector_PinHeader_1.27mm:PinHeader_1x01_P1.27mm_Vertical, symbol Connector:TestPoint
- added TP3: LowPass OUT, Connector_PinHeader_1.27mm:PinHeader_1x01_P1.27mm_Vertical, symbol Connector:TestPoint
- added TP4: HighPass OUT, Connector_PinHeader_1.27mm:PinHeader_1x01_P1.27mm_Vertical, symbol Connector:TestPoint
- added TP5: AMPLIFIER IN, Connector_PinHeader_1.27mm:PinHeader_1x01_P1.27mm_Vertical, symbol Connector:TestPoint
- added TP6: AMPLIFIER OUT, Connector_PinHeader_1.27mm:PinHeader_1x01_P1.27mm_Vertical, symbol Connector:TestPoint
- added TP7: IN -, Connector_PinHeader_1.27mm:PinHeader_1x01_P1.27mm_Vertical, symbol Connector:TestPoint
- added TP8: IN +, Connector_PinHeader_1.27mm:PinHeader_1x01_P1.27mm_Vertical, symbol Connector:TestPoint
- added TP9: AD623_OUT, Connector_PinHeader_1.27mm:PinHeader_1x01_P1.27mm_Vertical, symbol Connector:TestPoint
- added U4: AD623, Package_DIP:DIP-8_W7.62mm_LongPads, symbol Amplifier_Instrumentation:AD623
- added U5: TL071, Package_DIP:DIP-8_W7.62mm_LongPads, symbol Amplifier_Operational:TL071
- C1, C101, C2: footprint (none) -> Capacitor_THT:C_Rect_L7.2mm_W4.5mm_P5.00mm_FKS2_FKP2_MKS2_MKP2
- C102: footprint (none) -> Capacitor_THT:CP_Radial_D7.5mm_P2.50mm
- C103: value C -> 100n; footprint (none) -> Capacitor_THT:C_Rect_L7.2mm_W4.5mm_P5.00mm_FKS2_FKP2_MKS2_MKP2
- C104: value CP -> 47u; footprint (none) -> Capacitor_THT:CP_Radial_D7.5mm_P2.50mm
- C105: renamed from C?; value C -> 100n; footprint (none) -> Capacitor_THT:C_Rect_L7.2mm_W4.5mm_P5.00mm_FKS2_FKP2_MKS2_MKP2
- C106: renamed from C?; value CP -> 47u; footprint (none) -> Capacitor_THT:CP_Radial_D7.5mm_P2.50mm
- C3, C4: renamed from C?; footprint (none) -> Capacitor_THT:C_Rect_L7.2mm_W4.5mm_P5.00mm_FKS2_FKP2_MKS2_MKP2
- R1, R2, R3, R4: footprint (none) -> Resistor_THT:R_Axial_DIN0207_L6.3mm_D2.5mm_P10.16mm_Horizontal
- R10, R5, R6, R7, R8, R9: renamed from R?; footprint (none) -> Resistor_THT:R_Axial_DIN0207_L6.3mm_D2.5mm_P10.16mm_Horizontal
- U1, U2: footprint (none) -> Package_DIP:DIP-8_W7.62mm_LongPads
- U3: renamed from U?; footprint (none) -> Package_DIP:DIP-8_W7.62mm_LongPads
Connections:
- net AMP_OUT: now also TP6.1
- net GND: now also C107.2, C108.1, C109.2, C110.1, C111.2, C112.1, C5.2, C6.2, C7.2, C8.2, RV1.1, RV1.2, U4.4 (Vs-), U4.5 (Ref), U5.4 (V-); no longer R9.1, U1.4 (V-), U2.4 (V-), U3.4 (V-)
- net IN_AMP: now also JP2.2, JP22.2, TP5.1
- net IN_LP: now also R1.2, JP3.2, JP33.2, TP1.1; no longer C3.2
- net OUT_HP: now also JP3.1, JP33.1, TP4.1
- net OUT_LP: now also JP2.1, JP22.1, TP3.1
- net +15V renamed +12V
- new net: R9.1, RV1.3
- new net: R11.1, U4.1 (Rg)
- new net: TP7.1, U4.2 (-)
- new net: TP8.1, U4.3 (+)
- new net: U4.6, U5.3 (+)
- new net: R12.1, U4.8 (Rg)
- new net: R11.2, R12.2
- new net +5V: C5.1, C6.1, C7.1, C8.1, U4.7 (Vs+), U5.7 (V+)
- new net -12V: C107.1, C108.2, C109.1, C110.2, C111.1, C112.2, U1.4 (V-), U2.4 (V-), U3.4 (V-)
- new net IN: JP1.1, JP11.1, JP4.1, JP44.1, TP9.1, U5.2 (-), U5.6
- new net IN_HP: C3.2, JP1.2, JP11.2, JP4.2, JP44.2, TP2.1
- no-connect marks 0 -> 4
Other:
- moved on the sheet: C105, C106, R10, R9, U3
