File: ecg.kicad_pcb (KiCad board)
At the start: 2 copper layers, 110 x 99 mm, 66 parts, among them J1 Conn_01x03_Female, U1 TL072, U2 TL072, U3 TL071, U4 AD623, U5 TL071, U6 L7812, U7 L7912, U8 L7805

Commit message: pcb layout routed
Parts:
- moved C108 274.5 mm to (102.9, 109.2), turned to 90 degrees
- moved C105 271.2 mm to (96.5, 138.4), turned to 180 degrees
- moved JP2 269.4 mm to (120.7, 120.7)
- moved C106 269.3 mm to (95.2, 128.3), turned to 180 degrees
- moved C107 264.7 mm to (110.5, 105.4), turned to 270 degrees
- moved JP22 262.1 mm to (125.7, 120.7)
- moved U3 258.9 mm to (102.9, 127.0)
- moved TP3 250.5 mm to (130.8, 88.9)
- moved TP6 249.6 mm to (119.4, 128.3)
- moved C1 249.4 mm to (118.1, 109.2), turned to 90 degrees
- moved C111 248.2 mm to (101.6, 121.8), turned to 90 degrees
- moved RV1 246.4 mm to (115.6, 142.2)
- moved C101 245.9 mm to (108.0, 85.1)
- moved TP5 245.8 mm to (128.3, 128.3)
- moved JP3 232.7 mm to (143.5, 113.0), turned to 90 degrees
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Routing:
- net +12V: track 0.00 -> 226.5 mm, vias 0 -> 2
- net -12V: track 0.00 -> 213.6 mm, vias 0 -> 2
- net +5V: track 0.00 -> 101.8 mm
- net IN_HP: track 0.00 -> 85.6 mm, vias 0 -> 2
- net OUT_HP: track 0.00 -> 65.2 mm
- net IN: track 0.00 -> 62.5 mm
- net Net-(C10-Pad2): track 0.00 -> 52.2 mm
- net OUT_LP: track 0.00 -> 51.7 mm
- net IN_AMP: track 0.00 -> 36.0 mm
- net Net-(R7-Pad1): track 0.00 -> 34.5 mm, vias 0 -> 2
- net Net-(C2-Pad1): track 0.00 -> 34.3 mm, vias 0 -> 2
- net Net-(C4-Pad2): track 0.00 -> 31.6 mm
- net IN_LP: track 0.00 -> 30.7 mm
- net Net-(C1-Pad1): track 0.00 -> 27.8 mm
- net Net-(U4-Pad6): track 0.00 -> 27.7 mm
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- added copper zone on B.Cu, net GND
- added copper zone on F.Cu, net GND

Commit message: layout and fSilk added
Other:
- board text added: "ELECTROMEDICINA CLÍNICA"
- board text added: "HIGH PASS FILTER"
- board text added: "IES FEDERICA MONTSENY"
- board text added: "INPUT STAGE"
- board text added: "LOW PASS FILTER"
- board text added: "OUTPUT STAGE"
- board text added: "POWER SECTION"
- board text added: "Rev0"
- board text added: "SISTEMAS ELECTRÓNICOS Y FOTÓNICOS"
Changed lines of the file:
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@@
   (general
     (thickness 1.6)
-    (drawings 35)
+    (drawings 44)
     (tracks 290)
     (zones 0)
@@
     (descr "CP, Radial series, Radial, pin pitch=2.50mm, , diameter=7.5mm, Electrolytic Capacitor")
     (tags "CP Radial series Radial pin pitch 2.50mm  diameter 7.5mm Electrolytic Capacitor")
-    (fp_text reference C102 (at 1.25 -5) (layer F.SilkS)
+    (fp_text reference C102 (at 6.35 -3.81) (layer F.SilkS)
       (effects (font (size 1 1) (thickness 0.15)))
     )
@@
     )
   )
+  (gr_text "Rev0\n" (at 187.96 127) (layer F.SilkS)
+    (effects (font (size 1 1) (thickness 0.15)))
+  )
+  (gr_text "SISTEMAS ELECTRÓNICOS Y FOTÓNICOS\n" (at 165.1 144.145) (layer F.SilkS)
+    (effects (font (size 1.8 1.8) (thickness 0.15)))
+  )
+  (gr_text "ELECTROMEDICINA CLÍNICA\n" (at 158.75 140.97) (layer F.SilkS)
+    (effects (font (size 2 2) (thickness 0.15)))
+  )
+  (gr_text "IES FEDERICA MONTSENY\n" (at 157.48 137.16) (layer F.SilkS)
+    (effects (font (size 2 2) (thickness 0.15)))
+  )
+  (gr_text "POWER SECTION\n" (at 142.24 51.435) (layer F.SilkS)
+    (effects (font (size 1 1) (thickness 0.15)))
+  )
+  (gr_text "INPUT STAGE\n" (at 151.13 86.36) (layer F.SilkS)
+    (effects (font (size 1 1) (thickness 0.15)))
+  )
+  (gr_text "LOW PASS FILTER\n" (at 112.395 77.47) (layer F.SilkS)
+    (effects (font (size 1 1) (thickness 0.15)))
+  )
+  (gr_text "OUTPUT STAGE\n" (at 93.98 144.78) (layer F.SilkS)
+    (effects (font (size 1 1) (thickness 0.15)))
+  )
+  (gr_text "HIGH PASS FILTER\n" (at 146.05 127) (layer F.SilkS)
+    (effects (font (size 1 1) (thickness 0.15)))
+  )
   (gr_line (start 135.89 76.2) (end 135.89 113.03) (layer F.SilkS) (width 0.12))
